Commit message: added lidar to robot

File: catkin_ws/src/my_robot/urdf/my_robot.xacro (robot description, xacro)
@@ -97,4 +97,50 @@
         </visual>
     </link>
+    <link name="camera">
+        <inertial>
+            <mass value="0.1"/>
+            <origin xyz="0 0 0" rpy="0 0 0"/>
+            <inertia
+                    ixx="1e-6" ixy="0" ixz="0"
+                    iyy="1e-6" iyz="0"
+                    izz="1e-6"
+            />
+        </inertial>
+        <collision>
+            <origin xyz="0 0 0" rpy="0 0 0"/>
+            <geometry>
+                <box size="0.05 0.05 0.05"/>
+            </geometry>
+        </collision>
+        <visual>
+            <origin xyz="0 0 0" rpy="0 0 0"/>
+            <geometry>
+                <box size="0.05 0.05 0.05"/>
+            </geometry>
+        </visual>
+    </link>
+    <link name="hokuyo">
+        <inertial>
+            <mass value="1e-5"/>
+            <origin xyz="0 0 0" rpy="0 0 0"/>
+            <inertia
+                    ixx="1e-6" ixy="0" ixz="0"
+                    iyy="1e-6" iyz="0"
+                    izz="1e-6"
+            />
+        </inertial>
+        <collision>
+            <origin xyz="0 0 0" rpy="0 0 0"/>
+            <geometry>
+                <box size="0.1 0.1 0.1"/>
+            </geometry>
+        </collision>
+        <visual>
+            <origin xyz="0 0 0" rpy="0 0 0"/>
+            <geometry>
+                <mesh filename="package://my_robot/meshes/hokuyo.dae"/>
+            </geometry>
+        </visual>
+    </link>
     <!--Joints-->
     <joint name="robot_footprint_joint" type="fixed">
@@ -119,3 +165,15 @@
         <dynamics damping="1.0" friction="1.0"/>
     </joint>
+    <joint type="fixed" name="camera_joint">
+        <origin xyz="0.2 0 0" rpy="0 0 0"/>
+        <child link="camera"/>
+        <parent link="chassis"/>
+        <axis xyz="0 1 0" rpy="0 0 0"/>
+    </joint>
+    <joint type="fixed" name="hokuyo_joint">
+        <origin xyz="0.15 0 0.1" rpy="0 0 0"/>
+        <child link="hokuyo"/>
+        <parent link="chassis"/>
+        <axis xyz="0 1 0" rpy="0 0 0"/>
+    </joint>
 </robot>

Commit message: updated based on further feedback

File: catkin_ws/src/my_robot/urdf/my_robot.xacro (robot description, xacro)
@@ -25,6 +25,14 @@
                 <cylinder radius="0.1" length="0.05"/>
             </geometry>
-        </visual>
-    </link>
+            <material name="orange">
+                <color rgba="1.0 0.423529411765 0.0392156862745 1.0"/>
+            </material>
+        </visual>
+    </link>
+    <gazebo reference="left_wheel">
+        <material>
+            Gazebo/Orange
+        </material>
+    </gazebo>
     <link name="right_wheel">
         <inertial>
@@ -48,6 +56,14 @@
                 <cylinder radius="0.1" length="0.05"/>
             </geometry>
-        </visual>
-    </link>
+            <material name="orange">
+                <color rgba="1.0 0.423529411765 0.0392156862745 1.0"/>
+            </material>
+        </visual>
+    </link>
+    <gazebo reference="right_wheel">
+        <material>
+            Gazebo/Orange
+        </material>
+    </gazebo>
     <link name='chassis'>
         <pose>0 0 0.1 0 0 0</pose>
@@ -72,4 +88,7 @@
                 <box size=".4 .2 .1"/>
             </geometry>
+            <material name="black">
+                <color rgba="0.0 0.0 0.0 1.0"/>
+            </material>
         </visual>
         <collision name='back_caster_collision'>
@@ -98,4 +117,9 @@
         </visual>
     </link>
+    <gazebo reference="chassis">
+        <material>
+            Gazebo/Black
+        </material>
+    </gazebo>
     <link name="camera">
         <inertial>
@@ -119,6 +143,14 @@
                 <box size="0.05 0.05 0.05"/>
             </geometry>
-        </visual>
-    </link>
+            <material name="green">
+                <color rgba="0.0 0.8 0.0 1.0"/>
+            </material>
+        </visual>
+    </link>
+    <gazebo reference="camera">
+        <material>
+            Gazebo/Green
+        </material>
+    </gazebo>
     <link name="hokuyo">
         <inertial>
